File: sint-85/sint-85.kicad_sch (KiCad schematic)
At the start: 3 parts, among them U5 74LS138, U6 74LS32, U7 74LS00

Commit message: Updated port and bus connectors.
Parts:
- added J1: BUS, symbol Connector:Conn_01x47_Pin
- added J3: PORTS, symbol Connector_Generic:Conn_02x13_Counter_Clockwise
Connections:
- net A11: now also J1.30 (Pin_30)
- net A12: now also J1.29 (Pin_29)
- net A13: now also J1.28 (Pin_28)
- net A14: now also J1.27 (Pin_27)
- net A15: now also J1.26 (Pin_26)
- net GND: now also J1.2 (Pin_2), J3.1 (Pin_1), J3.26 (Pin_26)
- net ^RD: now also J1.45 (Pin_45)
- net Mem RD $0800 - $0FFF renamed J1.3 Mem RD $0800 - $0FFF
- net Mem RD $1000 - $17FF renamed J1.4 Mem RD $1000 - $17FF
- new net +5v: J1.1 (Pin_1), J3.2 (Pin_2), J3.25 (Pin_25)
- new net A0: J1.34 (Pin_34)
- new net A1: J1.35 (Pin_35)
- new net A10: J1.31 (Pin_31)
- new net A2: J1.36 (Pin_36)
- new net A3: J1.37 (Pin_37)
- new net A4: J1.38 (Pin_38)
- new net A5: J1.39 (Pin_39)
- new net A6: J1.40 (Pin_40)
- new net A7: J1.41 (Pin_41)
- new net A8: J1.33 (Pin_33)
- new net A9: J1.32 (Pin_32)
- new net ALE: J1.47 (Pin_47)
- new net CS  $2800-$2FFF: J1.6 (Pin_6)
- new net CS  $3000-$37FF: J1.5 (Pin_5)
- new net D0: J1.18 (Pin_18)
- new net D1: J1.19 (Pin_19)
- new net D2: J1.20 (Pin_20)
- new net D3: J1.21 (Pin_21)
- new net D4: J1.22 (Pin_22)
- new net D5: J1.23 (Pin_23)
- new net D6: J1.24 (Pin_24)
- new net D7: J1.25 (Pin_25)
- new net HLDA: J1.17 (Pin_17)
- new net HOLD: J1.16 (Pin_16)
- new net INTR: J1.11 (Pin_11)
- new net IO/^M: J1.44 (Pin_44)
- new net PA0: J3.13 (Pin_13)
- new net PA1: J3.14 (Pin_14)
- new net PA2: J3.12 (Pin_12)
- new net PA3: J3.15 (Pin_15)
- new net PA4: J3.11 (Pin_11)
- new net PA5: J3.16 (Pin_16)
- new net PA6: J3.10 (Pin_10)
- new net PA7: J3.17 (Pin_17)
- new net PB0: J3.9 (Pin_9)
- new net PB1: J3.18 (Pin_18)
- new net PB2: J3.8 (Pin_8)
- new net PB3: J3.19 (Pin_19)
- new net PB4: J3.7 (Pin_7)
- new net PB5: J3.20 (Pin_20)
- new net PB6: J3.6 (Pin_6)
- new net PB7: J3.21 (Pin_21)
- new net PC0: J3.5 (Pin_5)
- new net PC1: J3.22 (Pin_22)
- new net PC2: J3.4 (Pin_4)
- new net PC3: J3.23 (Pin_23)
- new net PC4: J3.3 (Pin_3)
- new net PC5: J3.24 (Pin_24)
- new net READY: J1.14 (Pin_14)
- new net RESET-OUT: J1.43 (Pin_43)
- new net RST 6.5: J1.13 (Pin_13)
- new net S0: J1.9 (Pin_9)
- new net S1: J1.12 (Pin_12)
- new net TIMER-IN (8155): J1.42 (Pin_42)
- new net ^CS $1800-$1FFF: J1.7 (Pin_7)
- new net ^CS *^RD $0800-$0FFF: J1.3 (Pin_3)
- new net ^CS *^RD $1000-$17FF: J1.4 (Pin_4)
- new net ^INTA: J1.10 (Pin_10)
- new net ^RESET-IN: J1.15 (Pin_15)
- new net ^WR: J1.46 (Pin_46)
- no-connect marks 0 -> 1
Other:
- moved on the sheet: U5, U6A, U6B, U6C, U6D, U7A, U7B, U7C, U7D
